File: oshpark/oshpark.kicad_pcb (KiCad board)
At the start: 2 copper layers, 0 parts

Commit message: Adjusted for jlcpcb.
Other:
- rule via_min_size: 0.508 -> 0.5588
Changed lines of the file:
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@@
     (via_size 1.016)
     (via_drill 0.762)
-    (via_min_size 0.508)
+    (via_min_size 0.5588)
     (via_min_drill 0.254)
     (uvia_size 1.016)
@@
     (uvia_min_size 0)
     (uvia_min_drill 0)
-    (edge_width 0.0508)
+    (edge_width 0.254)
     (segment_width 0.254)
     (pcb_text_width 0.3048)
     (pcb_text_size 1.524 1.524)
-    (mod_edge_width 0.127)
+    (mod_edge_width 0.2032)
     (mod_text_size 1.016 1.016)
-    (mod_text_width 0.1524)
+    (mod_text_width 0.2032)
     (pad_size 1.524 1.524)
     (pad_drill 0.762)
     (pad_to_mask_clearance 0.0508)
     (aux_axis_origin 0 0)
-    (visible_elements FFFFFF7F)
+    (visible_elements 7FFFFFFF)
     (pcbplotparams
       (layerselection 0x010fc_ffffffff)
